Commit message: Added base_footprint tf

File: urdf/bcr_bot.xacro (robot description, xacro)
@@ -50,5 +50,11 @@
     </xacro:if>
     <!-- ................................ BASE LINK .................................. -->
+    <link name="base_footprint"/>
     <link name="base_link"/>
+    <joint name="base_joint" type="fixed">
+        <parent link="base_footprint"/>
+        <child link="base_link"/>
+        <origin xyz="0.0 0 ${chassis_height/2 + traction_wheel_radius}" rpy="0 0 0.0" />
+    </joint>
     <link name="chassis_link">
         <collision>

File: urdf/gazebo.xacro (robot description, xacro)
@@ -18,5 +18,5 @@
             <wheel_separation>${traction_track_width+traction_wheel_width-0.01}</wheel_separation>
             <wheel_diameter>${2*traction_wheel_radius+0.01}</wheel_diameter>
-            <robot_base_frame>base_link</robot_base_frame>
+            <robot_base_frame>base_footprint</robot_base_frame>
             <max_wheel_torque>${traction_max_wheel_torque}</max_wheel_torque>
             <command_topic>cmd_vel</command_topic>
@@ -59,5 +59,5 @@
             <always_on>true</always_on>
             <update_rate>30.0</update_rate>
-            <body_name>base_link</body_name>
+            <body_name>base_footprint</body_name>
             <gaussian_noise>0.00</gaussian_noise>
             <frame_name>$(arg ground_truth_frame)</frame_name>

File: urdf/gz.xacro (robot description, xacro)
@@ -23,5 +23,5 @@
             </xacro:if>
             <frame_id>odom</frame_id>
-            <child_frame_id>base_link</child_frame_id>
+            <child_frame_id>base_footprint</child_frame_id>
         </plugin>
     </gazebo>
@@ -32,5 +32,5 @@
             name="ignition::gazebo::systems::OdometryPublisher">
             <odom_frame>odom</odom_frame>
-            <robot_base_frame>base_link</robot_base_frame>
+            <robot_base_frame>base_footprint</robot_base_frame>
             <odom_topic>$(arg wheel_odom_topic)</odom_topic>
             <tf_topic>/tf</tf_topic>
